File: Circuits/KiCad/Power-Clock/Power-Clock.kicad_pcb (KiCad board)
At the start: 2 copper layers, 104.1 x 104.1 mm, 50 parts, among them J1 BUS1, J2 BUS2, J3 Power (5V), SW1 Power, SW2 RESET, SW3 Single-step, SW4 Single-step, SW5 Turbo, U1 MCP100-450D, U2 555, U3 555, U4 74x04, U5 74x08, U6 555, U7 74x32, U8 74x08, U9 555, Y1 1 MHz

Commit message: Routed power & clock PCB
Parts:
- removed D5: LED, LED_THT:LED_D5.0mm
- removed R13: 1K, Resistor_THT:R_Axial_DIN0207_L6.3mm_D2.5mm_P7.62mm_Horizontal
- removed R14, R15: 330, Resistor_THT:R_Axial_DIN0207_L6.3mm_D2.5mm_P7.62mm_Horizontal
- removed U9: 555, Package_DIP:DIP-8_W7.62mm
- added C10: 100 nF, Capacitor_THT:C_Rect_L4.6mm_W3.0mm_P2.50mm_MKS02_FKP02, F.Cu at (40.6, 68.6)
- added C11: 1nF, Capacitor_THT:C_Rect_L4.6mm_W3.0mm_P2.50mm_MKS02_FKP02, F.Cu at (71.1, 63.5)
- added C9: 10nF, Capacitor_THT:C_Rect_L4.6mm_W2.0mm_P2.50mm_MKS02_FKP02, F.Cu at (87.9, 85.1)
- added F1: Polyfuse, Capacitor_THT:C_Disc_D9.0mm_W2.5mm_P5.00mm, F.Cu at (59.7, 49.5)
- C1: value 220µF -> 10nF; footprint Capacitor_THT:CP_Radial_D6.3mm_P2.50mm -> Capacitor_THT:C_Rect_L4.6mm_W2.0mm_P2.50mm_MKS02_FKP02
- C2: value 100 nF -> 100nF; footprint Capacitor_THT:C_Rect_L4.6mm_W3.0mm_P2.50mm_MKS02_FKP02 -> Capacitor_THT:C_Rect_L4.6mm_W2.0mm_P2.50mm_MKS02_FKP02
- C3: value 1uF -> 220µF; footprint Capacitor_THT:CP_Radial_D5.0mm_P2.50mm -> Capacitor_THT:CP_Radial_D6.3mm_P2.50mm
- C4, C5, C7, C8: value 10nF -> 100nF
- C6: value 100nF -> 10nF
- D2: value LED -> HALT
- D3: value LED -> POWER; footprint LED_THT:LED_D5.0mm -> LED_THT:LED_D5.0mm_Horizontal_O1.27mm_Z3.0mm
- D4: value LED -> STEP; footprint LED_THT:LED_D5.0mm -> LED_THT:LED_D5.0mm_Horizontal_O1.27mm_Z3.0mm
- J1: value BUS1 -> Power (5V); footprint Connector_PinHeader_2.54mm:PinHeader_2x20_P2.54mm_Vertical -> Connector_BarrelJack:BarrelJack_Horizontal
- J2: value BUS2 -> BUS1; footprint Connector_PinHeader_2.54mm:PinHeader_2x20_P2.54mm_Vertical -> Connector_PinSocket_2.54mm:PinSocket_2x20_P2.54mm_Vertical
- J3: value Power (5V) -> BUS2; footprint Connector_BarrelJack:BarrelJack_Horizontal -> Connector_PinSocket_2.54mm:PinSocket_2x20_P2.54mm_Vertical
- R10, R9: value 1K -> 330
- R11: value 330 -> 5K
- R12, R3, R6, R7: value 1K -> 5K
- R2: value 330 -> 100K
- R4: value 47K -> 330
- R5: value 1M -> 5K; footprint Potentiometer_THT:Potentiometer_Piher_PT-6-V_Vertical -> Resistor_THT:R_Axial_DIN0207_L6.3mm_D2.5mm_P7.62mm_Horizontal
- R8: value 1M -> 5K
- SW1: value Power -> Single-step; footprint Button_Switch_THT:SW_CuK_JS202011AQN_DPDT_Angled -> Button_Switch_THT:SW_Tactile_SKHH_Angled
- SW2: value RESET -> Power; footprint Button_Switch_THT:SW_Tactile_SKHH_Angled -> DM-02:Switch_DPST_Angled
- SW3: value Single-step -> CONTINUE; footprint 74xx-Computer-Footprints:SW_6mm_Tact -> Button_Switch_THT:SW_Tactile_SKHH_Angled
- SW4: footprint 74xx-Computer-Footprints:Switch -> DM-02:Slide-switch
- SW5: value Turbo -> RESET; footprint 74xx-Computer-Footprints:Switch -> Button_Switch_THT:SW_Tactile_SKHH_Angled
- U1: value MCP100-450D -> 555; footprint Package_TO_SOT_THT:TO-92 -> Package_DIP:DIP-8_W7.62mm
- U2: value 555 -> 74HCT04; footprint Package_DIP:DIP-8_W7.62mm -> Package_DIP:DIP-14_W7.62mm
- U4: value 74x04 -> 555; footprint Package_DIP:DIP-14_W7.62mm -> Package_DIP:DIP-8_W7.62mm
- U5: value 74x08 -> MCP100-450D; footprint Package_DIP:DIP-14_W7.62mm -> Package_TO_SOT_THT:TO-92
- U6: value 555 -> 74HCT08; footprint Package_DIP:DIP-8_W7.62mm -> Package_DIP:DIP-14_W7.62mm
- U7: value 74x32 -> 74HCT14
- U8: value 74x08 -> 74HCT32
- moved SW2 106.7 mm to (40.6, 50.8), turned to 90 degrees
- moved SW1 99.8 mm to (127.0, 86.4)
- moved J3 88.2 mm to (102.9, 124.5), turned to 270 degrees
- moved J2 86.4 mm to (102.9, 35.6)
- moved J1 77.7 mm to (38.7, 76.8), turned to 0 degrees
- moved R8 75.8 mm to (36.8, 57.1)
- moved SW5 74.4 mm to (30.5, 65.4), turned to 90 degrees
- moved C1 69.6 mm to (114.3, 85.1)
- moved R4 60.6 mm to (119.4, 54.4), turned to 90 degrees
- moved R1 58.3 mm to (103.6, 72.4), turned to 0 degrees
- moved U1 56.4 mm to (103.6, 77.5), turned to 0 degrees
- moved D1 56.1 mm to (49.5, 56.5)
- moved U8 53.2 mm to (37.6, 92.5)
- moved C2 52.7 mm to (100.1, 74.9), turned to 270 degrees
- moved C6 49.5 mm to (114.3, 108.0), turned to 90 degrees
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Connections:
- net Net-(J2-Pad10) renamed A0
- net Net-(J2-Pad12) renamed A1
- net Net-(J2-Pad14) renamed A2
- net Net-(J2-Pad15) renamed BUS1_1
- net Net-(J2-Pad16) renamed A3
- net Net-(J2-Pad17) renamed BUS1_2
- net Net-(J2-Pad18) renamed A4
- net Net-(J2-Pad19) renamed BUS1_3
- net Net-(J2-Pad20) renamed A5
- net Net-(J2-Pad21) renamed BUS1_4
- net Net-(J2-Pad22) renamed A6
- net Net-(J2-Pad23) renamed BUS1_5
- net Net-(J2-Pad24) renamed A7
- net Net-(J2-Pad25) renamed D0
- net Net-(J2-Pad26) renamed A8
- net Net-(J2-Pad27) renamed D1
- net Net-(J2-Pad28) renamed A9
- net Net-(J2-Pad29) renamed D2
- net Net-(J2-Pad30) renamed A10
- net Net-(J2-Pad31) renamed D3
- net Net-(J2-Pad32) renamed A11
- net Net-(J2-Pad33) renamed D4
- net Net-(J2-Pad34) renamed A12
- net Net-(J2-Pad35) renamed D5
- net Net-(J2-Pad36) renamed A13
- net Net-(J2-Pad37) renamed D6
- net Net-(J2-Pad38) renamed A14
- net Net-(J2-Pad39) renamed D7
- net Net-(J2-Pad4) renamed ~DEBUG_RESET
- net Net-(J2-Pad40) renamed A15
- C1 pad 1: +5V -> Net-(C1-Pad1)
- C1 pad 2: GND -> COMPUTER_GND
- C2 pad 1: GND -> Net-(C2-Pad1)
- C2 pad 2: +5V -> COMPUTER_GND
- C3 pad 1: Net-(C3-Pad1) -> COMPUTER_5V
- C3 pad 2: GND -> COMPUTER_GND
- C4 pad 1: Net-(C4-Pad1) -> COMPUTER_5V
- C4 pad 2: GND -> COMPUTER_GND
- C5 pad 1: Net-(C5-Pad1) -> COMPUTER_5V
- C5 pad 2: GND -> COMPUTER_GND
- C6 pad 2: GND -> COMPUTER_GND
- C7 pad 1: Net-(C7-Pad1) -> COMPUTER_5V
- C7 pad 2: GND -> COMPUTER_GND
- C8 pad 1: Net-(C8-Pad1) -> COMPUTER_5V
- C8 pad 2: GND -> COMPUTER_GND
- D1 pad 1: +5V -> COMPUTER_5V
- D1 pad 2: GND -> COMPUTER_GND
- D2 pad 2: ~RESET -> HALT
- D3 pad 2: STEP_EN -> ~RESET
- D4 pad 2: TURBO_EN -> STEP_EN
- J1 pad 1: GND -> Net-(J1-Pad1)
- J1 pad 2: +5V -> Net-(J1-Pad2)
- J1 pad 3: CLOCK1 -> (no net)
- J2 pad 1: HALT -> COMPUTER_GND
- J2 pad 11: Net-(J2-Pad11) -> CLOCK_ENABLE
- J2 pad 2: Net-(J2-Pad2) -> COMPUTER_5V
- J2 pad 3: CONTINUE -> CLOCK1
- J2 pad 5: Net-(J2-Pad5) -> CLOCK2
- J2 pad 6: Net-(J2-Pad6) -> ~RESET
- J2 pad 7: Net-(J2-Pad7) -> ~CLOCK1
- J2 pad 9: Net-(J2-Pad9) -> ~CLOCK2
- J3 pad 1: Net-(J3-Pad1) -> HALT
- J3 pad 2: Net-(J3-Pad2) -> BUS2_40
- J3 pad 3: (no net) -> CONTINUE
- R1 pad 1: ~RESET -> Net-(R1-Pad1)
- R1 pad 2: +5V -> COMPUTER_5V
- R10 pad 1: Net-(R10-Pad1) -> Net-(D4-Pad1)
- R10 pad 2: +5V -> COMPUTER_GND
- R11 pad 1: Net-(D3-Pad1) -> COMPUTER_GND
- R11 pad 2: GND -> Net-(R11-Pad2)
- R12 pad 1: Net-(R12-Pad1) -> COMPUTER_5V
- R12 pad 2: +5V -> CLOCK_ENABLE
- R2 pad 1: +5V -> COMPUTER_5V
- R2 pad 2: Net-(D2-Pad1) -> Net-(C2-Pad1)
- R3 pad 2: +5V -> COMPUTER_5V
- R4 pad 1: Net-(C3-Pad1) -> Net-(D2-Pad1)
- R4 pad 2: Net-(R4-Pad2) -> COMPUTER_GND
- R5 pad 2: Net-(R5-Pad2) -> COMPUTER_5V
- R6 pad 1: Net-(R3-Pad1) -> Net-(R6-Pad1)
- R6 pad 2: Net-(R5-Pad2) -> COMPUTER_5V
- R7 pad 1: Net-(R7-Pad1) -> HALT
- R7 pad 2: +5V -> COMPUTER_5V
- R8 pad 1: +5V -> ~RESET
- R8 pad 2: Net-(C6-Pad1) -> COMPUTER_5V
- R9 pad 1: Net-(R9-Pad1) -> COMPUTER_GND
- R9 pad 2: +5V -> Net-(D3-Pad1)
- SW1 pad 1: Net-(J3-Pad2) -> COMPUTER_GND
- SW1 pad 2: GND -> Net-(R1-Pad1)
- SW2 pad 1: GND -> Net-(J1-Pad2)
- SW2 pad 2: ~RESET -> COMPUTER_GND
- SW3 pad 1: GND -> COMPUTER_5V
- SW3 pad 2: Net-(R7-Pad1) -> CONTINUE
- SW4 pad 1: Net-(R9-Pad1) -> Net-(R3-Pad1)
- SW4 pad 2: GND -> COMPUTER_GND
- SW4 pad 3: Net-(R10-Pad1) -> Net-(R5-Pad1)
- SW5 pad 1: Net-(R12-Pad1) -> COMPUTER_GND
- SW5 pad 2: GND -> ~RESET
- U1 pad 1: ~RESET -> COMPUTER_GND
- U1 pad 2: +5V -> Net-(R1-Pad1)
- U1 pad 3: GND -> CLK_STEP
- U2 pad 1: GND -> CONTINUE
- U2 pad 2: Net-(C3-Pad1) -> Net-(R6-Pad1)
- U2 pad 3: CLK_VARIABLE -> STEP_EN
- U2 pad 4: +5V -> Net-(U2-Pad4)
- U2 pad 5: Net-(C4-Pad1) -> HALT
- U2 pad 6: Net-(C3-Pad1) -> Net-(U2-Pad6)
- U2 pad 7: Net-(R3-Pad1) -> COMPUTER_GND
- U2 pad 8: +5V -> (no net)
- U3 pad 1: GND -> COMPUTER_GND
- U3 pad 2: Net-(R7-Pad1) -> Net-(R3-Pad1)
- U3 pad 3: CLK_STEP -> STEP_EN
- U3 pad 4: +5V -> Net-(R5-Pad1)
- U3 pad 5: Net-(C5-Pad1) -> Net-(C6-Pad1)
- U3 pad 6: Net-(C6-Pad1) -> COMPUTER_GND
- U3 pad 7: Net-(C6-Pad1) -> Net-(U3-Pad7)
- U3 pad 8: +5V -> COMPUTER_5V
- U4 pad 1: STEP_EN -> COMPUTER_GND
- U4 pad 2: Net-(U4-Pad2) -> Net-(R6-Pad1)
- U4 pad 3: HALT -> Net-(R11-Pad2)
- U4 pad 4: Net-(U4-Pad4) -> HALT
- U4 pad 5: TURBO_EN -> Net-(C9-Pad1)
- U4 pad 6: Net-(U4-Pad6) -> COMPUTER_GND
- U4 pad 7: GND -> Net-(U4-Pad7)
- U4 pad 8: (no net) -> COMPUTER_5V
- U5 pad 1: STEP_EN -> ~RESET
- U5 pad 2: CLK_STEP -> COMPUTER_5V
- U5 pad 3: STEP_EN -> COMPUTER_GND
- U6 pad 1: GND -> CLK_STEP
- U6 pad 2: Net-(R9-Pad1) -> STEP_EN
- U6 pad 3: STEP_EN -> Net-(U6-Pad3)
- U6 pad 4: Net-(R10-Pad1) -> Net-(U2-Pad4)
- U6 pad 5: Net-(C7-Pad1) -> CLK_OSC
- U6 pad 6: GND -> Net-(U6-Pad6)
- U6 pad 7: Net-(U6-Pad7) -> COMPUTER_GND
- U6 pad 8: +5V -> Net-(U6-Pad13)
- U7 pad 1: Net-(U5-Pad8) -> CLOCK1
- U7 pad 10: Net-(U7-Pad10) -> (no net)
- U7 pad 14: +5V -> COMPUTER_5V
- U7 pad 2: STEP_EN -> ~CLOCK1
- U7 pad 3: Net-(U7-Pad3) -> CLOCK1
- U7 pad 4: Net-(U5-Pad11) -> Net-(C11-Pad2)
- U7 pad 5: Net-(U4-Pad6) -> Net-(C11-Pad2)
- U7 pad 6: Net-(U7-Pad6) -> CLOCK2
- U7 pad 7: GND -> COMPUTER_GND
- U7 pad 8: Net-(U7-Pad8) -> ~CLOCK2
- U7 pad 9: Net-(U7-Pad9) -> CLOCK2
- U8 pad 1: Net-(U5-Pad6) -> Net-(U2-Pad6)
- U8 pad 10: Net-(U4-Pad4) -> (no net)
- U8 pad 14: +5V -> COMPUTER_5V
- U8 pad 2: CLK_TURBO -> Net-(R11-Pad2)
- U8 pad 3: Net-(U7-Pad10) -> Net-(U6-Pad10)
- U8 pad 4: Net-(U7-Pad3) -> Net-(U6-Pad3)
- U8 pad 5: Net-(U7-Pad6) -> Net-(U6-Pad6)
- U8 pad 6: Net-(U7-Pad9) -> Net-(U6-Pad9)
- U8 pad 7: GND -> COMPUTER_GND
- U8 pad 8: CLOCK1 -> (no net)
- U8 pad 9: Net-(U7-Pad8) -> (no net)
- Y1 pad 1: +5V -> COMPUTER_5V
- Y1 pad 2: GND -> COMPUTER_GND
- Y1 pad 3: CLK_TURBO -> CLK_OSC
Routing:
- net COMPUTER_GND: track 0.00 -> 424.3 mm
- net COMPUTER_5V: track 0.00 -> 292.0 mm
- net HALT: track 0.00 -> 147.0 mm
- net CONTINUE: track 0.00 -> 135.2 mm
- net ~RESET: track 0.00 -> 116.5 mm
- net STEP_EN: track 0.00 -> 103.5 mm
- net CLOCK1: track 0.00 -> 89.9 mm
- net CLOCK_ENABLE: track 0.00 -> 77.4 mm, vias 0 -> 1
- net CLK_OSC: track 0.00 -> 69.4 mm
- net Net-(U6-Pad10): track 0.00 -> 68.3 mm
- net Net-(U6-Pad9): track 0.00 -> 53.6 mm
- net Net-(R11-Pad2): track 0.00 -> 44.8 mm
- net CLOCK2: track 0.00 -> 41.8 mm
- net Net-(U6-Pad6): track 0.00 -> 40.8 mm
- net Net-(U6-Pad3): track 0.00 -> 40.6 mm
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- added copper zone on B.Cu, net COMPUTER_GND
- added copper zone on F.Cu, net COMPUTER_GND
Other:
- outline, holes or cut-outs redrawn
- board text added: "1.1"
- board text added: "1.2"
- board text added: "1.3"
- board text added: "1.4"
- board text added: "1.5"
- board text added: "2.10"
- board text added: "2.11"
- board text added: "2.12"
- board text added: "2.13"
- board text added: "2.14"
- board text added: "2.15"
- board text added: "2.16"
- board text added: "2.17"
- board text added: "2.18"
- board text added: "2.19"
- board text added: "2.20"
- board text added: "2.21"
- board text added: "2.22"
- board text added: "2.23"
- board text added: "2.24"
- board text added: "2.25"
- board text added: "2.26"
- board text added: "2.27"
- board text added: "2.28"
- board text added: "2.29"
- board text added: "2.3"
- board text added: "2.30"
- board text added: "2.31"
- board text added: "2.32"
- board text added: "2.33"
- board text added: "2.34"
- board text added: "2.35"
- board text added: "2.36"
- board text added: "2.37"
- board text added: "2.38"
- board text added: "2.39"
- board text added: "2.4"
- board text added: "2.40"
- board text added: "2.5"
- board text added: "2.6"
- board text added: "2.7"
- board text added: "2.8"
- board text added: "2.9"
- board text added: "5V"
- board text added: "A0"
- board text added: "A1"
- board text added: "A10"
- board text added: "A11"
- board text added: "A12"
- board text added: "A13"
- board text added: "A14"
- board text added: "A15"
- board text added: "A2"
- board text added: "A3"
- board text added: "A4"
- board text added: "A5"
- board text added: "A6"
- board text added: "A7"
- board text added: "A8"
- board text added: "A9"
- board text added: "CLK_EN"
- board text added: "CLOCK1"
- board text added: "CLOCK2"
- board text added: "CONT"
- board text added: "D0"
- board text added: "D1"
- board text added: "D2"
- board text added: "D3"
- board text added: "D4"
- board text added: "D5"
- board text added: "D6"
- board text added: "D7"
- board text added: "GND"
- board text added: "HALT"
- board text added: "NC4"
- board text added: "NC5"
- board text added: "~CLOCK1"
- board text added: "~CLOCK2"
- board text added: "~DRST"
- board text added: "~RST"

Commit message: Documentation
Changed lines of the file:
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@@
   (page A4)
   (layers
-    (0 F.Cu signal)
-    (31 B.Cu signal)
+    (0 F.Cu signal hide)
+    (31 B.Cu signal hide)
     (32 B.Adhes user hide)
     (33 F.Adhes user hide)
@@
       (effects (font (size 1 1) (thickness 0.15)))
     )
-    (fp_text value 74HCT08 (at 3.81 17.57) (layer F.Fab)
+    (fp_text value 74HCT08 (at 4.064 7.62 90) (layer F.SilkS)
       (effects (font (size 1 1) (thickness 0.15)))
     )
@@
       (effects (font (size 1 1) (thickness 0.15)))
     )
-    (fp_text value MCP100-450D (at 1.27 2.79 90) (layer F.Fab)
-      (effects (font (size 1 1) (thickness 0.15)))
+    (fp_text value MCP100-450D (at 1.27 2.79 90) (layer B.SilkS)
+      (effects (font (size 1 1) (thickness 0.15)) (justify mirror))
     )
     (fp_arc (start 1.27 0) (end 1.27 -2.6) (angle 135) (layer F.SilkS) (width 0.12))
@@
       (effects (font (size 1 1) (thickness 0.15)))
     )
-    (fp_text value 555 (at 3.81 9.95) (layer F.Fab)
+    (fp_text value 555 (at 3.81 3.81) (layer F.SilkS)
       (effects (font (size 1 1) (thickness 0.15)))
     )
@@
       (effects (font (size 1 1) (thickness 0.15)))
     )
-    (fp_text value 74HCT04 (at 3.81 17.57) (layer F.Fab)
+    (fp_text value 74HCT04 (at 3.81 7.874 90) (layer F.SilkS)
       (effects (font (size 1 1) (thickness 0.15)))
     )
@@
       (effects (font (size 1 1) (thickness 0.15)))
     )
-    (fp_text value 555 (at 3.81 9.95) (layer F.Fab)
+    (fp_text value 555 (at 3.81 3.81) (layer F.SilkS)
       (effects (font (size 1 1) (thickness 0.15)))
     )
@@
       (effects (font (size 1 1) (thickness 0.15)))
     )
-    (fp_text value "Power (5V)" (at -6.2 -5.5) (layer F.Fab)
+    (fp_text value "Power (5V)" (at -6.2 -5.5) (layer F.SilkS)
       (effects (font (size 1 1) (thickness 0.15)))
     )
@@
       (effects (font (size 1 1) (thickness 0.15)))
     )
-    (fp_text value "100 nF" (at 1.25 2.75) (layer F.Fab)
-      (effects (font (size 1 1) (thickness 0.15)))
+    (fp_text value "100 nF" (at 1.27 2.54) (layer B.SilkS)
+      (effects (font (size 1 1) (thickness 0.15)) (justify mirror))
     )
     (fp_text user %R (at 1.25 0) (layer F.Fab)
@@
       (effects (font (size 1 1) (thickness 0.15)))
     )
-    (fp_text value 220µF (at 1.25 4.4 90) (layer F.Fab)
+    (fp_text value 220µF (at 1.25 4.4 90) (layer F.SilkS)
       (effects (font (size 1 1) (thickness 0.15)))
     )
@@
       (effects (font (size 1 1) (thickness 0.15)))
     )
-    (fp_text value "1 MHz" (at 3.81 3.74 90) (layer F.Fab)
+    (fp_text value "1 MHz" (at 3.81 -3.556 270) (layer F.SilkS)
       (effects (font (size 1 1) (thickness 0.15)))
     )
@@
       (effects (font (size 1 1) (thickness 0.15)))
     )
-    (fp_text value 74HCT14 (at 3.81 17.57) (layer F.Fab)
+    (fp_text value 74HCT14 (at 3.81 7.62 90) (layer F.SilkS)
       (effects (font (size 1 1) (thickness 0.15)))
     )
@@
       (effects (font (size 1 1) (thickness 0.15)))
     )
-    (fp_text value 74HCT32 (at 3.81 17.57) (layer F.Fab)
+    (fp_text value 74HCT32 (at 3.683 7.874 90) (layer F.SilkS)
       (effects (font (size 1 1) (thickness 0.15)))
     )
@@
       (effects (font (size 1 1) (thickness 0.15)))
     )
-    (fp_text value 555 (at 3.81 9.95) (layer F.Fab)
-      (effects (font (size 1 1) (thickness 0.15)))
-    )
+    (fp_text value 555 (at 3.683 3.81 180) (layer F.SilkS)
+      (effects (font (size 1 1) (thickness 0.15)))
+    )

Commit message: -
Parts:
- removed J2: BUS1, Connector_PinSocket_2.54mm:PinSocket_2x20_P2.54mm_Vertical
- removed J3: BUS2, Connector_PinSocket_2.54mm:PinSocket_2x20_P2.54mm_Vertical
- added BUS1: Conn_02x32_Odd_Even, Connector_PinSocket_2.54mm:PinSocket_2x32_P2.54mm_Vertical, F.Cu at (252.7, 39.4)
- added BUS2: Conn_02x32_Odd_Even, Connector_PinSocket_2.54mm:PinSocket_2x32_P2.54mm_Vertical, F.Cu at (252.7, 135.9)
- moved H3 138.9 mm to (264.2, 137.2)
- moved H4 138.5 mm to (264.2, 35.6)
- moved H2 131.3 mm to (162.6, 137.2)
- moved H1 130.9 mm to (162.6, 35.6)
Routing:
- net COMPUTER_GND: track 424.3 -> 0.00 mm
- net COMPUTER_5V: track 292.0 -> 0.00 mm
- net HALT: track 147.0 -> 0.00 mm
- net CONTINUE: track 135.2 -> 0.00 mm
- net ~RESET: track 116.5 -> 0.00 mm
- net STEP_EN: track 103.5 -> 0.00 mm
- net CLOCK1: track 89.9 -> 0.00 mm
- net CLOCK_ENABLE: track 77.4 -> 0.00 mm, vias 1 -> 0
- net CLK_OSC: track 69.4 -> 0.00 mm
- net Net-(U6-Pad10): track 68.3 -> 0.00 mm
- net Net-(U6-Pad9): track 53.6 -> 0.00 mm
- net Net-(R11-Pad2): track 44.8 -> 0.00 mm
- net CLOCK2: track 41.8 -> 0.00 mm
- net Net-(U6-Pad6): track 40.8 -> 0.00 mm
- net Net-(U6-Pad3): track 40.6 -> 0.00 mm
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- removed copper zone on B.Cu, net COMPUTER_GND
- removed copper zone on F.Cu, net COMPUTER_GND
Other:
- board size 104.1 x 104.1 mm -> 121.9 x 121.9 mm
- board text added: "-"
- board text added: "ALUFUNC0"
- board text added: "ALUFUNC1"
- board text added: "ALUFUNC2"
- board text added: "ALUFUNC3"
- board text added: "ALUFUNC4"
- board text added: "BTN_CONTINUE"
- board text added: "BTN_RESET"
- board text added: "BTN_STEP"
- board text added: "BTN_STEP_ENA"
- board text added: "CLOCK_ENABLE"
- board text added: "CLOCK_PH0"
- board text added: "CLOCK_PH1"
- board text added: "CLOCK_PH2"
- board text added: "CLOCK_PH3"
- board text added: "DATA0"
- board text added: "DATA1"
- board text added: "DATA2"
- board text added: "DATA3"
- board text added: "DATA4"
- board text added: "DATA5"
- board text added: "DATA6"
- board text added: "DATA7"
- board text added: "DESIGNED BY RUUD VAN FALIER"
- board text added: "DM-02 8-Bit Computer"
- board text added: "DM-02 | Power & Clock | Revision 2"
- board text added: "FETCH_done"
- board text added: "FLAGS0"
- board text added: "FLAGS1"
- board text added: "FLAGS2"
- board text added: "FLAGS3"
- board text added: "INSTR0"
- board text added: "INSTR1"
- board text added: "INSTR2"
- board text added: "INSTR3"
- board text added: "INSTR4"
- board text added: "INSTR5"
- board text added: "INSTR6"
- board text added: "INSTR7"
- board text added: "IO_load"
- board text added: "IO_out"
- board text added: "PC_inc"
- board text added: "STK_dec"
- board text added: "STK_inc"
- board text added: "TSTATE0"
- board text added: "TSTATE1"
- board text added: "TSTATE2"
- board text added: "TSTATE3"
- board text added: "TSTATE_reset"
- board text added: "https://dutchmaker.com"
- board text added: "~ALU_load"
- board text added: "~ALU_out"
- board text added: "~A_load"
- board text added: "~A_out"
- board text added: "~B_load"
- board text added: "~B_out"
- board text added: "~C_load"
- board text added: "~C_out"
- board text added: "~FCLR_c"
- board text added: "~FCLR_z"
- board text added: "~FSET_c"
- board text added: "~FSET_z"
- board text added: "~F_load"
- board text added: "~F_out"
- board text added: "~H_load"
- board text added: "~H_out"
- board text added: "~IR_load"
- board text added: "~L_load"
- board text added: "~L_out"
- board text added: "~MAR_H_load"
- board text added: "~MAR_L_load"
- board text added: "~MAR_inc"
- board text added: "~MEM_load"
- board text added: "~MEM_out"
- board text added: "~PC_H_load"
- board text added: "~PC_H_out"
- board text added: "~PC_L_load"
- board text added: "~PC_L_out"
- board text added: "~PC_MAR_trans"
- board text added: "~STK_H_load"
- board text added: "~STK_H_out"
- board text added: "~STK_L_load"
- board text added: "~STK_L_out"
- board text added: "~STK_MAR_trans"
- board text removed: "1.1"
- board text removed: "1.2"
- board text removed: "1.3"
- board text removed: "1.4"
- board text removed: "1.5"
- board text removed: "2.10"
- board text removed: "2.11"
- board text removed: "2.12"
- board text removed: "2.13"
- board text removed: "2.14"
- board text removed: "2.15"
- board text removed: "2.16"
- board text removed: "2.17"
- board text removed: "2.18"
- board text removed: "2.19"
- board text removed: "2.20"
- board text removed: "2.21"
- board text removed: "2.22"
- board text removed: "2.23"
- board text removed: "2.24"
- board text removed: "2.25"
- board text removed: "2.26"
- board text removed: "2.27"
- board text removed: "2.28"
- board text removed: "2.29"
- board text removed: "2.3"
- board text removed: "2.30"
- board text removed: "2.31"
- board text removed: "2.32"
- board text removed: "2.33"
- board text removed: "2.34"
- board text removed: "2.35"
- board text removed: "2.36"
- board text removed: "2.37"
- board text removed: "2.38"
- board text removed: "2.39"
- board text removed: "2.4"
- board text removed: "2.40"
- board text removed: "2.5"
- board text removed: "2.6"
- board text removed: "2.7"
- board text removed: "2.8"
- board text removed: "2.9"
- board text removed: "CLK_EN"
- board text removed: "CLOCK1"
- board text removed: "CLOCK2"
- board text removed: "CONT"
- board text removed: "D0"
- board text removed: "D1"
- board text removed: "D2"
- board text removed: "D3"
- board text removed: "D4"
- board text removed: "D5"
- board text removed: "D6"
- board text removed: "D7"
- board text removed: "NC4"
- board text removed: "NC5"
- board text removed: "Power & Clock | Revision 1"
- board text removed: "~CLOCK1"
- board text removed: "~CLOCK2"
- board text removed: "~DRST"
- board text removed: "~RST"
